Commit message: Add lh or rh prefix to links and joints

File: lh_robothand_a0_description/urdf/lh_robothand_a0.urdf (robot description, URDF)
Before this commit: robot lh_robothand_a0, 16 links, 15 joints
Links:
- removed link FF1_Link
- removed link FF2_Link
- removed link FF3_Link
- removed link LF1_Link
- removed link LF2_Link
- removed link LF3_Link
- removed link MF1_Link
- removed link MF2_Link
- removed link MF3_Link
- removed link RF1_Link
- removed link RF2_Link
- removed link RF3_Link
- removed link TH1_Link
- removed link TH2_Link
- removed link TH3_Link
- removed link base_link
- added link lh_FF1_Link, mass 0.00833003074086424; collision mesh filename=package://lh_robothand_a0_description/meshes/FF1_Link.STL; visual mesh filename=package://lh_robothand_a0_description/meshes/FF1_Link.STL
- added link lh_FF2_Link, mass 0.00216268861976196; collision mesh filename=package://lh_robothand_a0_description/meshes/FF2_Link.STL; visual mesh filename=package://lh_robothand_a0_description/meshes/FF2_Link.STL
- added link lh_FF3_Link, mass 0.00337032712997865; collision mesh filename=package://lh_robothand_a0_description/meshes/FF3_Link.STL; visual mesh filename=package://lh_robothand_a0_description/meshes/FF3_Link.STL
- added link lh_LF1_Link, mass 0.0074874409052179; collision mesh filename=package://lh_robothand_a0_description/meshes/LF1_Link.STL; visual mesh filename=package://lh_robothand_a0_description/meshes/LF1_Link.STL
- added link lh_LF2_Link, mass 0.0020406717952195; collision mesh filename=package://lh_robothand_a0_description/meshes/LF2_Link.STL; visual mesh filename=package://lh_robothand_a0_description/meshes/LF2_Link.STL
- added link lh_LF3_Link, mass 0.0024374814930342; collision mesh filename=package://lh_robothand_a0_description/meshes/LF3_Link.STL; visual mesh filename=package://lh_robothand_a0_description/meshes/LF3_Link.STL
- added link lh_MF1_Link, mass 0.0097069421206806; collision mesh filename=package://lh_robothand_a0_description/meshes/MF1_Link.STL; visual mesh filename=package://lh_robothand_a0_description/meshes/MF1_Link.STL
- added link lh_MF2_Link, mass 0.00228824509732534; collision mesh filename=package://lh_robothand_a0_description/meshes/MF2_Link.STL; visual mesh filename=package://lh_robothand_a0_description/meshes/MF2_Link.STL
- added link lh_MF3_Link, mass 0.00336556031844797; collision mesh filename=package://lh_robothand_a0_description/meshes/MF3_Link.STL; visual mesh filename=package://lh_robothand_a0_description/meshes/MF3_Link.STL
- added link lh_RF1_Link, mass 0.0083300368382922; collision mesh filename=package://lh_robothand_a0_description/meshes/RF1_Link.STL; visual mesh filename=package://lh_robothand_a0_description/meshes/RF1_Link.STL
- added link lh_RF2_Link, mass 0.00216268864685091; collision mesh filename=package://lh_robothand_a0_description/meshes/RF2_Link.STL; visual mesh filename=package://lh_robothand_a0_description/meshes/RF2_Link.STL
- added link lh_RF3_Link, mass 0.00336561552955153; collision mesh filename=package://lh_robothand_a0_description/meshes/RF3_Link.STL; visual mesh filename=package://lh_robothand_a0_description/meshes/RF3_Link.STL
- added link lh_TH1_Link, mass 0.0376965566076027; collision mesh filename=package://lh_robothand_a0_description/meshes/TH1_Link.STL; visual mesh filename=package://lh_robothand_a0_description/meshes/TH1_Link.STL
- added link lh_TH2_Link, mass 0.00973663443524222; collision mesh filename=package://lh_robothand_a0_description/meshes/TH2_Link.STL; visual mesh filename=package://lh_robothand_a0_description/meshes/TH2_Link.STL
- added link lh_TH3_Link, mass 0.0049133; collision mesh filename=package://lh_robothand_a0_description/meshes/TH3_Link.STL; visual mesh filename=package://lh_robothand_a0_description/meshes/TH3_Link.STL
- added link lh_base_link, mass 0.262848373649471; collision mesh filename=package://lh_robothand_a0_description/meshes/base_link.STL; visual mesh filename=package://lh_robothand_a0_description/meshes/base_link.STL
Joints:
- removed joint FF1
- removed joint FF2
- removed joint FF3
- removed joint LF1
- removed joint LF2
- removed joint LF3
- removed joint MF1
- removed joint MF2
- removed joint MF3
- removed joint RF1
- removed joint RF2
- removed joint RF3
- removed joint TH1
- removed joint TH2
- removed joint TH3
- added joint lh_FF1: type revolute, parent lh_base_link, child lh_FF1_Link, origin xyz=-0.02808 0.12467 -0.0032197 rpy=0 0 0, axis -1 0 0, limit lower=-1.57 upper=0 effort=1 velocity=-0.5, mimic joint=lh_FF2 multiplier=1.8 offset=0
- added joint lh_FF2: type revolute, parent lh_FF1_Link, child lh_FF2_Link, origin xyz=0.0002 0.044498 0.00044206 rpy=0 0 0, axis -1 0 0, limit lower=-1.57 upper=0 effort=1 velocity=-0.5, mimic joint=lh_FF3 multiplier=1.8 offset=0
- added joint lh_FF3: type revolute, parent lh_FF2_Link, child lh_FF3_Link, origin xyz=0 0.024491 0.00065357 rpy=0 0 0, axis -1 0 0, limit lower=-1 upper=0 effort=1 velocity=-0.5
- added joint lh_LF1: type revolute, parent lh_base_link, child lh_LF1_Link, origin xyz=0.02722 0.12067 -0.0012197 rpy=0 0 0, axis -1 0 0, limit lower=-1.57 upper=0 effort=1 velocity=-0.5, mimic joint=lh_LF2 multiplier=1.8 offset=0
- added joint lh_LF2: type revolute, parent lh_LF1_Link, child lh_LF2_Link, origin xyz=0 0.040097 -0.00037218 rpy=0 0 0, axis -1 0 0, limit lower=-1.57 upper=0 effort=1 velocity=-0.5, mimic joint=lh_LF3 multiplier=1.8 offset=0
- added joint lh_LF3: type revolute, parent lh_LF2_Link, child lh_LF3_Link, origin xyz=0 0.02198 0.00094344 rpy=0 0 0, axis -1 0 0, limit lower=-1 upper=0 effort=1 velocity=-0.5
- added joint lh_MF1: type revolute, parent lh_base_link, child lh_MF1_Link, origin xyz=-0.0094801 0.12667 -0.0047197 rpy=0 0 0, axis -1 0 0, limit lower=-1.57 upper=0 effort=1 velocity=-0.5, mimic joint=lh_MF2 multiplier=1.8 offset=0
- added joint lh_MF2: type revolute, parent lh_MF1_Link, child lh_MF2_Link, origin xyz=0 0.047487 0.0011335 rpy=0 0 0, axis -1 0 0, limit lower=-1.57 upper=0 effort=1 velocity=-0.5, mimic joint=lh_MF3 multiplier=1.8 offset=0
- added joint lh_MF3: type revolute, parent lh_MF2_Link, child lh_MF3_Link, origin xyz=0 0.026482 0.00098138 rpy=0 0 0, axis -1 0 0, limit lower=-1 upper=0 effort=1 velocity=-0.5
- added joint lh_RF1: type revolute, parent lh_base_link, child lh_RF1_Link, origin xyz=0.0090199 0.12467 -0.0032197 rpy=0 0 0, axis -1 0 0, limit lower=-1.57 upper=0 effort=1 velocity=-0.5, mimic joint=lh_RF2 multiplier=1.8 offset=0
- added joint lh_RF2: type revolute, parent lh_RF1_Link, child lh_RF2_Link, origin xyz=0.0002 0.0445 0.00020578 rpy=0 0 0, axis -1 0 0, limit lower=-1.57 upper=0 effort=1 velocity=-0.5, mimic joint=lh_RF3 multiplier=1.8 offset=0
- added joint lh_RF3: type revolute, parent lh_RF2_Link, child lh_RF3_Link, origin xyz=0 0.024497 0.00039909 rpy=0 0 0, axis -1 0 0, limit lower=-1 upper=0 effort=1 velocity=-0.5
- added joint lh_TH1: type revolute, parent lh_base_link, child lh_TH1_Link, origin xyz=-0.024843 0.061673 0.0085578 rpy=0 0 1.5708, axis -1 0 0, limit lower=0 upper=1 effort=1 velocity=0.5, mimic joint=lh_TH2 multiplier=-1.8 offset=0
- added joint lh_TH2: type revolute, parent lh_TH1_Link, child lh_TH2_Link, origin xyz=0.029023 0.041949 0.02497 rpy=0 -1.0472 -1.5708, axis 1 0 0, limit lower=-0.65 upper=0 effort=1 velocity=-0.5, mimic joint=lh_TH3 multiplier=1.8 offset=0
- added joint lh_TH3: type revolute, parent lh_TH2_Link, child lh_TH3_Link, origin xyz=0 0.030805 0.02225 rpy=0 0 0, axis 1 0 0, limit lower=-0.79 upper=0 effort=1 velocity=0.5

File: lh_robothand_a0_description/urdf/lh_robothand_a0.xacro (robot description, xacro)
@@ -6,5 +6,5 @@
   name="lh_robothand_a0" xmlns:xacro="http://www.ros.org/wiki/xacro">
   <link
-    name="base_link">
+    name="lh_base_link">
     <inertial>
       <origin
@@ -46,5 +46,5 @@
   </link>
   <link
-    name="LF1_Link">
+    name="lh_LF1_Link">
     <inertial>
       <origin
@@ -86,5 +86,5 @@
   </link>
   <joint
-    name="LF1"
+    name="lh_LF1"
     type="revolute">
     <origin
@@ -92,7 +92,7 @@
       rpy="0 0 0" />
     <parent
-      link="base_link" />
-    <child
-      link="LF1_Link" />
+      link="lh_base_link" />
+    <child
+      link="lh_LF1_Link" />
     <axis
       xyz="-1 0 0" />
@@ -106,10 +106,10 @@
       friction="0.1" />
     <mimic
-      joint="LF2"
+      joint="lh_LF2"
       multiplier="1.8"
       offset="0" />
   </joint>
   <link
-    name="LF2_Link">
+    name="lh_LF2_Link">
     <inertial>
       <origin
@@ -151,5 +151,5 @@
   </link>
   <joint
-    name="LF2"
+    name="lh_LF2"
     type="revolute">
     <origin
@@ -157,7 +157,7 @@
       rpy="0 0 0" />
     <parent
-      link="LF1_Link" />
-    <child
-      link="LF2_Link" />
+      link="lh_LF1_Link" />
+    <child
+      link="lh_LF2_Link" />
     <axis
       xyz="-1 0 0" />
@@ -171,10 +171,10 @@
       friction="0.1" />
     <mimic
-      joint="LF3"
+      joint="lh_LF3"
       multiplier="1.8"
       offset="0" />
   </joint>
   <link
-    name="LF3_Link">
+    name="lh_LF3_Link">
     <inertial>
       <origin
@@ -216,5 +216,5 @@
   </link>
   <joint
-    name="LF3"
+    name="lh_LF3"
     type="revolute">
     <origin
@@ -222,7 +222,7 @@
       rpy="0 0 0" />
     <parent
-      link="LF2_Link" />
-    <child
-      link="LF3_Link" />
+      link="lh_LF2_Link" />
+    <child
+      link="lh_LF3_Link" />
     <axis
       xyz="-1 0 0" />
@@ -237,5 +237,5 @@
   </joint>
   <link
-    name="RF1_Link">
+    name="lh_RF1_Link">
     <inertial>
       <origin
@@ -277,5 +277,5 @@
   </link>
   <joint
-    name="RF1"
+    name="lh_RF1"
     type="revolute">
     <origin
@@ -283,7 +283,7 @@
       rpy="0 0 0" />
     <parent
-      link="base_link" />
-    <child
-      link="RF1_Link" />
+      link="lh_base_link" />
+    <child
+      link="lh_RF1_Link" />
     <axis
       xyz="-1 0 0" />
@@ -297,10 +297,10 @@
       friction="0.1" />
     <mimic
-      joint="RF2"
+      joint="lh_RF2"
       multiplier="1.8"
       offset="0" />
   </joint>
   <link
-    name="RF2_Link">
+    name="lh_RF2_Link">
     <inertial>
       <origin
@@ -342,5 +342,5 @@
   </link>
   <joint
-    name="RF2"
+    name="lh_RF2"
     type="revolute">
     <origin
@@ -348,7 +348,7 @@
       rpy="0 0 0" />
     <parent
-      link="RF1_Link" />
-    <child
-      link="RF2_Link" />
+      link="lh_RF1_Link" />
+    <child
+      link="lh_RF2_Link" />
     <axis
       xyz="-1 0 0" />
@@ -362,10 +362,10 @@
       friction="0.1" />
     <mimic
-      joint="RF3"
+      joint="lh_RF3"
       multiplier="1.8"
       offset="0" />
   </joint>
   <link
-    name="RF3_Link">
+    name="lh_RF3_Link">
     <inertial>
       <origin
@@ -407,5 +407,5 @@
   </link>
   <joint
-    name="RF3"
+    name="lh_RF3"
     type="revolute">
     <origin
@@ -413,7 +413,7 @@
       rpy="0 0 0" />
     <parent
-      link="RF2_Link" />
-    <child
-      link="RF3_Link" />
+      link="lh_RF2_Link" />
+    <child
+      link="lh_RF3_Link" />
     <axis
       xyz="-1 0 0" />
@@ -428,5 +428,5 @@
   </joint>
   <link
-    name="MF1_Link">
+    name="lh_MF1_Link">
     <inertial>
       <origin
@@ -468,5 +468,5 @@
   </link>
   <joint
-    name="MF1"
+    name="lh_MF1"
     type="revolute">
     <origin
@@ -474,7 +474,7 @@
       rpy="0 0 0" />
     <parent
-      link="base_link" />
-    <child
-      link="MF1_Link" />
+      link="lh_base_link" />
+    <child
+      link="lh_MF1_Link" />
     <axis
       xyz="-1 0 0" />
@@ -488,10 +488,10 @@
       friction="0.1" />
     <mimic
-      joint="MF2"
+      joint="lh_MF2"
       multiplier="1.8"
       offset="0" />
   </joint>
   <link
-    name="MF2_Link">
+    name="lh_MF2_Link">
     <inertial>
       <origin
@@ -533,5 +533,5 @@
   </link>
   <joint
-    name="MF2"
+    name="lh_MF2"
     type="revolute">
     <origin
@@ -539,7 +539,7 @@
       rpy="0 0 0" />
     <parent
-      link="MF1_Link" />
-    <child
-      link="MF2_Link" />
+      link="lh_MF1_Link" />
+    <child
+      link="lh_MF2_Link" />
     <axis
       xyz="-1 0 0" />
@@ -553,10 +553,10 @@
       friction="0.1" />
     <mimic
-      joint="MF3"
+      joint="lh_MF3"
       multiplier="1.8"
       offset="0" />
   </joint>
   <link
-    name="MF3_Link">
+    name="lh_MF3_Link">
     <inertial>
       <origin
@@ -598,5 +598,5 @@
   </link>
   <joint
-    name="MF3"
+    name="lh_MF3"
     type="revolute">
     <origin
@@ -604,7 +604,7 @@
       rpy="0 0 0" />
     <parent
-      link="MF2_Link" />
-    <child
-      link="MF3_Link" />
+      link="lh_MF2_Link" />
+    <child
+      link="lh_MF3_Link" />
     <axis
       xyz="-1 0 0" />
@@ -619,5 +619,5 @@
   </joint>
   <link
-    name="FF1_Link">
+    name="lh_FF1_Link">
     <inertial>
       <origin
@@ -659,5 +659,5 @@
   </link>
   <joint
-    name="FF1"
+    name="lh_FF1"
     type="revolute">
     <origin
@@ -665,7 +665,7 @@
       rpy="0 0 0" />
     <parent
-      link="base_link" />
-    <child
-      link="FF1_Link" />
+      link="lh_base_link" />
+    <child
+      link="lh_FF1_Link" />
     <axis
       xyz="-1 0 0" />
@@ -679,10 +679,10 @@
       friction="0.1" />
     <mimic
-      joint="FF2"
+      joint="lh_FF2"
       multiplier="1.8"
       offset="0" />
   </joint>
   <link
-    name="FF2_Link">
+    name="lh_FF2_Link">
     <inertial>
       <origin
@@ -724,5 +724,5 @@
   </link>
   <joint
-    name="FF2"
+    name="lh_FF2"
     type="revolute">
     <origin
@@ -730,7 +730,7 @@
       rpy="0 0 0" />
     <parent
-      link="FF1_Link" />
-    <child
-      link="FF2_Link" />
+      link="lh_FF1_Link" />
+    <child
+      link="lh_FF2_Link" />
     <axis
       xyz="-1 0 0" />
@@ -744,10 +744,10 @@
       friction="0.1" />
     <mimic
-      joint="FF3"
+      joint="lh_FF3"
       multiplier="1.8"
       offset="0" />
   </joint>
   <link
-    name="FF3_Link">
+    name="lh_FF3_Link">
     <inertial>
       <origin
@@ -789,5 +789,5 @@
   </link>
   <joint
-    name="FF3"
+    name="lh_FF3"
     type="revolute">
     <origin
@@ -795,7 +795,7 @@
       rpy="0 0 0" />
     <parent
-      link="FF2_Link" />
-    <child
-      link="FF3_Link" />
+      link="lh_FF2_Link" />
+    <child
+      link="lh_FF3_Link" />
     <axis
       xyz="-1 0 0" />
@@ -810,5 +810,5 @@
   </joint>
   <link
-    name="TH1_Link">
+    name="lh_TH1_Link">
     <inertial>
       <origin
@@ -850,5 +850,5 @@
   </link>
   <joint
-    name="TH1"
+    name="lh_TH1"
     type="revolute">
     <origin
@@ -856,7 +856,7 @@
       rpy="0 0 1.5708" />
     <parent
-      link="base_link" />
-    <child
-      link="TH1_Link" />
+      link="lh_base_link" />
+    <child
+      link="lh_TH1_Link" />
     <axis
       xyz="-1 0 0" />
@@ -870,10 +870,10 @@
       friction="0.1" />
     <mimic
-      joint="TH2"
+      joint="lh_TH2"
       multiplier="-1.8"
       offset="0" />
   </joint>
   <link
-    name="TH2_Link">
+    name="lh_TH2_Link">
     <inertial>
       <origin
@@ -915,5 +915,5 @@
   </link>
   <joint
-    name="TH2"
+    name="lh_TH2"
     type="revolute">
     <origin
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
File: rh_robothand_a0_description/urdf/rh_robothand_a0.urdf (robot description, URDF)
Before this commit: robot rh_robothand_a0, 16 links, 15 joints
Links:
- removed link FF1_Link
- removed link FF2_Link
- removed link FF3_Link
- removed link LF1_Link
- removed link LF2_Link
- removed link LF3_Link
- removed link MF1_Link
- removed link MF2_Link
- removed link MF3_Link
- removed link RF1_Link
- removed link RF2_Link
- removed link RF3_Link
- removed link TH1_Link
- removed link TH2_Link
- removed link TH3_Link
- removed link base_link
- added link rh_FF1_Link, mass 0.00847314272707745; collision mesh filename=package://rh_robothand_a0_description/meshes/FF1_Link.STL; visual mesh filename=package://rh_robothand_a0_description/meshes/FF1_Link.STL
- added link rh_FF2_Link, mass 0.00216268848240887; collision mesh filename=package://rh_robothand_a0_description/meshes/FF2_Link.STL; visual mesh filename=package://rh_robothand_a0_description/meshes/FF2_Link.STL
- added link rh_FF3_Link, mass 0.00337011127275863; collision mesh filename=package://rh_robothand_a0_description/meshes/FF3_Link.STL; visual mesh filename=package://rh_robothand_a0_description/meshes/FF3_Link.STL
- added link rh_LF1_Link, mass 0.0076305557950374; collision mesh filename=package://rh_robothand_a0_description/meshes/LF1_Link.STL; visual mesh filename=package://rh_robothand_a0_description/meshes/LF1_Link.STL
- added link rh_LF2_Link, mass 0.00204066265868655; collision mesh filename=package://rh_robothand_a0_description/meshes/LF2_Link.STL; visual mesh filename=package://rh_robothand_a0_description/meshes/LF2_Link.STL
- added link rh_LF3_Link, mass 0.00243753133684015; collision mesh filename=package://rh_robothand_a0_description/meshes/LF3_Link.STL; visual mesh filename=package://rh_robothand_a0_description/meshes/LF3_Link.STL
- added link rh_MF1_Link, mass 0.00985006169632293; collision mesh filename=package://rh_robothand_a0_description/meshes/MF1_Link.STL; visual mesh filename=package://rh_robothand_a0_description/meshes/MF1_Link.STL
- added link rh_MF2_Link, mass 0.00228824564195563; collision mesh filename=package://rh_robothand_a0_description/meshes/MF2_Link.STL; visual mesh filename=package://rh_robothand_a0_description/meshes/MF2_Link.STL
- added link rh_MF3_Link, mass 0.00336503153264149; collision mesh filename=package://rh_robothand_a0_description/meshes/MF3_Link.STL; visual mesh filename=package://rh_robothand_a0_description/meshes/MF3_Link.STL
- added link rh_RF1_Link, mass 0.00847314272707846; collision mesh filename=package://rh_robothand_a0_description/meshes/RF1_Link.STL; visual mesh filename=package://rh_robothand_a0_description/meshes/RF1_Link.STL
- added link rh_RF2_Link, mass 0.00216268866837306; collision mesh filename=package://rh_robothand_a0_description/meshes/RF2_Link.STL; visual mesh filename=package://rh_robothand_a0_description/meshes/RF2_Link.STL
- added link rh_RF3_Link, mass 0.00337008134334144; collision mesh filename=package://rh_robothand_a0_description/meshes/RF3_Link.STL; visual mesh filename=package://rh_robothand_a0_description/meshes/RF3_Link.STL
- added link rh_TH1_Link, mass 0.0376918113829352; collision mesh filename=package://rh_robothand_a0_description/meshes/TH1_Link.STL; visual mesh filename=package://rh_robothand_a0_description/meshes/TH1_Link.STL
- added link rh_TH2_Link, mass 0.00931281919634013; collision mesh filename=package://rh_robothand_a0_description/meshes/TH2_Link.STL; visual mesh filename=package://rh_robothand_a0_description/meshes/TH2_Link.STL
- added link rh_TH3_Link, mass 0.00491308218882966; collision mesh filename=package://rh_robothand_a0_description/meshes/TH3_Link.STL; visual mesh filename=package://rh_robothand_a0_description/meshes/TH3_Link.STL
- added link rh_base_link, mass 0.264420980793865; collision mesh filename=package://rh_robothand_a0_description/meshes/base_link.STL; visual mesh filename=package://rh_robothand_a0_description/meshes/base_link.STL
Joints:
- removed joint FF1
- removed joint FF2
- removed joint FF3
- removed joint LF1
- removed joint LF2
- removed joint LF3
- removed joint MF1
- removed joint MF2
- removed joint MF3
- removed joint RF1
- removed joint RF2
- removed joint RF3
- removed joint TH1
- removed joint TH2
- removed joint TH3
- added joint rh_FF1: type revolute, parent rh_base_link, child rh_FF1_Link, origin xyz=-0.124667710792653 0.0283801051279036 -0.00321967793702234 rpy=3.14159265358979 0 1.57079632679489, axis -1 0 0, limit lower=-1.57 upper=0 effort=1 velocity=-0.5, mimic joint=rh_FF2 multiplier=1.8 offset=0
- added joint rh_FF2: type revolute, parent rh_FF1_Link, child rh_FF2_Link, origin xyz=0 -0.0444999999936168 -0.000238749430078741 rpy=3.14159265358979 0 3.14159265358979, axis 1 0 0, limit lower=-1.57 upper=0 effort=1 velocity=-0.5, mimic joint=rh_FF3 multiplier=1.8 offset=0
- added joint rh_FF3: type revolute, parent rh_FF2_Link, child rh_FF3_Link, origin xyz=0 -0.024496145135367 0.000434595797305956 rpy=0 0 0, axis 1 0 0, limit lower=-1 upper=0 effort=1 velocity=0.5
- added joint rh_LF1: type revolute, parent rh_base_link, child rh_LF1_Link, origin xyz=-0.120667710792653 -0.0276205870569372 -0.0012196779370232 rpy=-3.14159265358979 0 1.5707963267949, axis -1 0 0, limit lower=-1.57 upper=0 effort=1 velocity=-0.5, mimic joint=rh_LF2 multiplier=1.8 offset=0
- added joint rh_LF2: type revolute, parent rh_LF1_Link, child rh_LF2_Link, origin xyz=0 -0.0400984606909391 -0.000233749430079859 rpy=3.14159265358979 0 3.14159265358979, axis 1 0 0, limit lower=-1.57 upper=0 effort=1 velocity=-0.5, mimic joint=rh_LF3 multiplier=1.8 offset=0
- added joint rh_LF3: type revolute, parent rh_LF2_Link, child rh_LF3_Link, origin xyz=4.99999999999043E-05 -0.0219426636355103 0.00158729725598191 rpy=0 0 0, axis 1 0 0, limit lower=-1 upper=0 effort=1 velocity=-0.5
- added joint rh_MF1: type revolute, parent rh_base_link, child rh_MF1_Link, origin xyz=-0.126667710792653 0.00957941294306249 -0.00471967793702235 rpy=3.14159265358979 0 1.5707963267949, axis -1 0 0, limit lower=-1.57 upper=0 effort=1 velocity=-0.5, mimic joint=rh_MF2 multiplier=1.8 offset=0
- added joint rh_MF2: type revolute, parent rh_MF1_Link, child rh_MF2_Link, origin xyz=0 -0.0474999999936168 -0.000238749430078922 rpy=3.14159265358979 0 -3.14159265358979, axis 1 0 0, limit lower=-1.57 upper=0 effort=1 velocity=-0.5, mimic joint=rh_MF3 multiplier=1.8 offset=0
- added joint rh_MF3: type revolute, parent rh_MF2_Link, child rh_MF3_Link, origin xyz=0 -0.0264999981219051 0 rpy=0 0 0, axis 1 0 0, limit lower=-1 upper=0 effort=1 velocity=-0.5
- added joint rh_RF1: type revolute, parent rh_base_link, child rh_RF1_Link, origin xyz=-0.124667710792653 -0.00861989487209627 -0.00321967793702238 rpy=-3.14159265358979 0 1.5707963267949, axis -1 0 0, limit lower=-1.57 upper=0 effort=1 velocity=-0.5, mimic joint=rh_RF2 multiplier=1.8 offset=0
- added joint rh_RF2: type revolute, parent rh_RF1_Link, child rh_RF2_Link, origin xyz=0 -0.0444999999936167 -0.000238749430078784 rpy=3.14159265358979 0 3.14159265358979, axis 1 0 0, limit lower=-1.57 upper=0 effort=1 velocity=-0.5, mimic joint=rh_RF3 multiplier=1.8 offset=0
- added joint rh_RF3: type revolute, parent rh_RF2_Link, child rh_RF3_Link, origin xyz=-0.000200000000000051 -0.024496145135367 0.000434595797305881 rpy=0 0 0, axis 1 0 0, limit lower=-1 upper=0 effort=1 velocity=-0.5
- added joint rh_TH1: type revolute, parent rh_base_link, child rh_TH1_Link, origin xyz=-0.0584729772678924 0.0248430195360303 0.00855783635789703 rpy=0 0 -3.14159265358979, axis -1 0 0, limit lower=0 upper=1 effort=1 velocity=0.5, mimic joint=rh_TH2 multiplier=-1.8 offset=0
- added joint rh_TH2: type revolute, parent rh_TH1_Link, child rh_TH2_Link, origin xyz=0.031184 -0.043702 0.024365 rpy=0 -1.0472 1.5708, axis -1 0 0, limit lower=-0.65 upper=0 effort=1 velocity=-0.5, mimic joint=rh_TH3 multiplier=1.8 offset=0
- added joint rh_TH3: type revolute, parent rh_TH2_Link, child rh_TH3_Link, origin xyz=0 -0.0308049280341684 0.0222498631188981 rpy=0 0 0, axis -1 0 0, limit lower=-0.79 upper=0 effort=1 velocity=0.5
