Commit message: Add lh or rh prefix to links and joints

File: rh_robothand_a0_description/urdf/rh_robothand_a0.xacro (robot description, xacro)
@@ -6,5 +6,5 @@
   name="rh_robothand_a0" xmlns:xacro="http://www.ros.org/wiki/xacro">
   <link
-    name="base_link">
+    name="rh_base_link">
     <inertial>
       <origin
@@ -32,5 +32,5 @@
         name="">
         <color
-          rgba="0 0.501960784313725 0 1" />
+          rgba="0.898039215686275 0.917647058823529 0.929411764705882 1" />
       </material>
     </visual>
@@ -46,5 +46,5 @@
   </link>
   <link
-    name="LF1_Link">
+    name="rh_LF1_Link">
     <inertial>
       <origin
@@ -86,5 +86,5 @@
   </link>
   <joint
-    name="LF1"
+    name="rh_LF1"
     type="revolute">
     <origin
@@ -92,7 +92,7 @@
       rpy="-3.14159265358979 0 1.5707963267949" />
     <parent
-      link="base_link" />
-    <child
-      link="LF1_Link" />
+      link="rh_base_link" />
+    <child
+      link="rh_LF1_Link" />
     <axis
       xyz="-1 0 0" />
@@ -106,10 +106,10 @@
       friction="0.1" />
     <mimic
-      joint="LF2"
+      joint="rh_LF2"
       multiplier="1.8"
       offset="0" />
   </joint>
   <link
-    name="LF2_Link">
+    name="rh_LF2_Link">
     <inertial>
       <origin
@@ -151,5 +151,5 @@
   </link>
   <joint
-    name="LF2"
+    name="rh_LF2"
     type="revolute">
     <origin
@@ -157,7 +157,7 @@
       rpy="3.14159265358979 0 3.14159265358979" />
     <parent
-      link="LF1_Link" />
-    <child
-      link="LF2_Link" />
+      link="rh_LF1_Link" />
+    <child
+      link="rh_LF2_Link" />
     <axis
       xyz="1 0 0" />
@@ -171,10 +171,10 @@
       friction="0.1" />
     <mimic
-      joint="LF3"
+      joint="rh_LF3"
       multiplier="1.8"
       offset="0" />
   </joint>
   <link
-    name="LF3_Link">
+    name="rh_LF3_Link">
     <inertial>
       <origin
@@ -216,5 +216,5 @@
   </link>
   <joint
-    name="LF3"
+    name="rh_LF3"
     type="revolute">
     <origin
@@ -222,7 +222,7 @@
       rpy="0 0 0" />
     <parent
-      link="LF2_Link" />
-    <child
-      link="LF3_Link" />
+      link="rh_LF2_Link" />
+    <child
+      link="rh_LF3_Link" />
     <axis
       xyz="1 0 0" />
@@ -237,5 +237,5 @@
   </joint>
   <link
-    name="RF1_Link">
+    name="rh_RF1_Link">
     <inertial>
       <origin
@@ -277,5 +277,5 @@
   </link>
   <joint
-    name="RF1"
+    name="rh_RF1"
     type="revolute">
     <origin
@@ -283,7 +283,7 @@
       rpy="-3.14159265358979 0 1.5707963267949" />
     <parent
-      link="base_link" />
-    <child
-      link="RF1_Link" />
+      link="rh_base_link" />
+    <child
+      link="rh_RF1_Link" />
     <axis
       xyz="-1 0 0" />
@@ -297,10 +297,10 @@
       friction="0.1" />
     <mimic
-      joint="RF2"
+      joint="rh_RF2"
       multiplier="1.8"
       offset="0" />
   </joint>
   <link
-    name="RF2_Link">
+    name="rh_RF2_Link">
     <inertial>
       <origin
@@ -342,5 +342,5 @@
   </link>
   <joint
-    name="RF2"
+    name="rh_RF2"
     type="revolute">
     <origin
@@ -348,7 +348,7 @@
       rpy="3.14159265358979 0 3.14159265358979" />
     <parent
-      link="RF1_Link" />
-    <child
-      link="RF2_Link" />
+      link="rh_RF1_Link" />
+    <child
+      link="rh_RF2_Link" />
     <axis
       xyz="1 0 0" />
@@ -362,10 +362,10 @@
       friction="0.1" />
     <mimic
-      joint="RF3"
+      joint="rh_RF3"
       multiplier="1.8"
       offset="0" />
   </joint>
   <link
-    name="RF3_Link">
+    name="rh_RF3_Link">
     <inertial>
       <origin
@@ -407,5 +407,5 @@
   </link>
   <joint
-    name="RF3"
+    name="rh_RF3"
     type="revolute">
     <origin
@@ -413,7 +413,7 @@
       rpy="0 0 0" />
     <parent
-      link="RF2_Link" />
-    <child
-      link="RF3_Link" />
+      link="rh_RF2_Link" />
+    <child
+      link="rh_RF3_Link" />
     <axis
       xyz="1 0 0" />
@@ -428,5 +428,5 @@
   </joint>
   <link
-    name="MF1_Link">
+    name="rh_MF1_Link">
     <inertial>
       <origin
@@ -468,5 +468,5 @@
   </link>
   <joint
-    name="MF1"
+    name="rh_MF1"
     type="revolute">
     <origin
@@ -474,7 +474,7 @@
       rpy="3.14159265358979 0 1.5707963267949" />
     <parent
-      link="base_link" />
-    <child
-      link="MF1_Link" />
+      link="rh_base_link" />
+    <child
+      link="rh_MF1_Link" />
     <axis
       xyz="-1 0 0" />
@@ -488,10 +488,10 @@
       friction="0.1" />
     <mimic
-      joint="MF2"
+      joint="rh_MF2"
       multiplier="1.8"
       offset="0" />
   </joint>
   <link
-    name="MF2_Link">
+    name="rh_MF2_Link">
     <inertial>
       <origin
@@ -533,5 +533,5 @@
   </link>
   <joint
-    name="MF2"
+    name="rh_MF2"
     type="revolute">
     <origin
@@ -539,7 +539,7 @@
       rpy="3.14159265358979 0 -3.14159265358979" />
     <parent
-      link="MF1_Link" />
-    <child
-      link="MF2_Link" />
+      link="rh_MF1_Link" />
+    <child
+      link="rh_MF2_Link" />
     <axis
       xyz="1 0 0" />
@@ -553,10 +553,10 @@
       friction="0.1" />
     <mimic
-      joint="MF3"
+      joint="rh_MF3"
       multiplier="1.8"
       offset="0" />
   </joint>
   <link
-    name="MF3_Link">
+    name="rh_MF3_Link">
     <inertial>
       <origin
@@ -598,5 +598,5 @@
   </link>
   <joint
-    name="MF3"
+    name="rh_MF3"
     type="revolute">
     <origin
@@ -604,7 +604,7 @@
       rpy="0 0 0" />
     <parent
-      link="MF2_Link" />
-    <child
-      link="MF3_Link" />
+      link="rh_MF2_Link" />
+    <child
+      link="rh_MF3_Link" />
     <axis
       xyz="1 0 0" />
@@ -619,5 +619,5 @@
   </joint>
   <link
-    name="FF1_Link">
+    name="rh_FF1_Link">
     <inertial>
       <origin
@@ -659,5 +659,5 @@
   </link>
   <joint
-    name="FF1"
+    name="rh_FF1"
     type="revolute">
     <origin
@@ -665,7 +665,7 @@
       rpy="3.14159265358979 0 1.57079632679489" />
     <parent
-      link="base_link" />
-    <child
-      link="FF1_Link" />
+      link="rh_base_link" />
+    <child
+      link="rh_FF1_Link" />
     <axis
       xyz="-1 0 0" />
@@ -679,10 +679,10 @@
       friction="0.1" />
     <mimic
-      joint="FF2"
+      joint="rh_FF2"
       multiplier="1.8"
       offset="0" />
   </joint>
   <link
-    name="FF2_Link">
+    name="rh_FF2_Link">
     <inertial>
       <origin
@@ -724,5 +724,5 @@
   </link>
   <joint
-    name="FF2"
+    name="rh_FF2"
     type="revolute">
     <origin
@@ -730,7 +730,7 @@
       rpy="3.14159265358979 0 3.14159265358979" />
     <parent
-      link="FF1_Link" />
-    <child
-      link="FF2_Link" />
+      link="rh_FF1_Link" />
+    <child
+      link="rh_FF2_Link" />
     <axis
       xyz="1 0 0" />
@@ -744,10 +744,10 @@
       friction="0.1" />
     <mimic
-      joint="FF3"
+      joint="rh_FF3"
       multiplier="1.8"
       offset="0" />
   </joint>
   <link
-    name="FF3_Link">
+    name="rh_FF3_Link">
     <inertial>
       <origin
@@ -789,5 +789,5 @@
   </link>
   <joint
-    name="FF3"
+    name="rh_FF3"
     type="revolute">
     <origin
@@ -795,7 +795,7 @@
       rpy="0 0 0" />
     <parent
-      link="FF2_Link" />
-    <child
-      link="FF3_Link" />
+      link="rh_FF2_Link" />
+    <child
+      link="rh_FF3_Link" />
     <axis
       xyz="1 0 0" />
@@ -810,5 +810,5 @@
   </joint>
   <link
-    name="TH1_Link">
+    name="rh_TH1_Link">
     <inertial>
       <origin
@@ -850,5 +850,5 @@
   </link>
   <joint
-    name="TH1"
+    name="rh_TH1"
     type="revolute">
     <origin
@@ -856,7 +856,7 @@
       rpy="0 0 -3.14159265358979" />
     <parent
-      link="base_link" />
-    <child
-      link="TH1_Link" />
+      link="rh_base_link" />
+    <child
+      link="rh_TH1_Link" />
     <axis
       xyz="-1 0 0" />
@@ -870,10 +870,10 @@
       friction="0.1" />
     <mimic
-      joint="TH2"
+      joint="rh_TH2"
       multiplier="-1.8"
       offset="0" />
   </joint>
   <link
-    name="TH2_Link">
+    name="rh_TH2_Link">
     <inertial>
       <origin
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
Commit message: Use primitive and VERY rough collision geometries

File: lh_robothand_a0_description/urdf/lh_robothand_a0.urdf (robot description, URDF)
Before this commit: robot lh_robothand_a0, 16 links, 15 joints
Links:
- link lh_FF1_Link: geometry visual mesh filename=package://lh_robothand_a0_description/meshes/FF1_Link.STL
- link lh_FF2_Link: geometry visual mesh filename=package://lh_robothand_a0_description/meshes/FF2_Link.STL
- link lh_FF3_Link: geometry visual mesh filename=package://lh_robothand_a0_description/meshes/FF3_Link.STL
- link lh_LF1_Link: geometry visual mesh filename=package://lh_robothand_a0_description/meshes/LF1_Link.STL
- link lh_LF2_Link: geometry visual mesh filename=package://lh_robothand_a0_description/meshes/LF2_Link.STL
- link lh_LF3_Link: geometry visual mesh filename=package://lh_robothand_a0_description/meshes/LF3_Link.STL
- link lh_MF1_Link: geometry visual mesh filename=package://lh_robothand_a0_description/meshes/MF1_Link.STL
- link lh_MF2_Link: geometry visual mesh filename=package://lh_robothand_a0_description/meshes/MF2_Link.STL
- link lh_MF3_Link: geometry visual mesh filename=package://lh_robothand_a0_description/meshes/MF3_Link.STL
- link lh_RF1_Link: geometry visual mesh filename=package://lh_robothand_a0_description/meshes/RF1_Link.STL
- link lh_RF2_Link: geometry visual mesh filename=package://lh_robothand_a0_description/meshes/RF2_Link.STL
- link lh_RF3_Link: geometry visual mesh filename=package://lh_robothand_a0_description/meshes/RF3_Link.STL
- link lh_TH1_Link: geometry visual mesh filename=package://lh_robothand_a0_description/meshes/TH1_Link.STL
- link lh_TH2_Link: geometry visual mesh filename=package://lh_robothand_a0_description/meshes/TH2_Link.STL
- link lh_TH3_Link: geometry visual mesh filename=package://lh_robothand_a0_description/meshes/TH3_Link.STL
- link lh_base_link: geometry collision box size=0.08 0.22 0.05; visual mesh filename=package://lh_robothand_a0_description/meshes/base_link.STL

File: lh_robothand_a0_description/urdf/lh_robothand_a0.xacro (robot description, xacro)
@@ -37,9 +37,8 @@
     <collision>
       <origin
-        xyz="0 0 0"
-        rpy="0 0 0" />
-      <geometry>
-        <mesh
-          filename="package://lh_robothand_a0_description/meshes/base_link.STL" />
+        xyz="0 0.11 0"
+        rpy="0 0 0" />
+      <geometry>
+        <box size="0.08 0.22 0.05"/>
       </geometry>
     </collision>
@@ -75,5 +74,5 @@
       </material>
     </visual>
-    <collision>
+    <!-- <collision>
       <origin
         xyz="0 0 0"
@@ -83,5 +82,5 @@
           filename="package://lh_robothand_a0_description/meshes/LF1_Link.STL" />
       </geometry>
-    </collision>
+    </collision> -->
   </link>
   <joint
@@ -140,5 +139,5 @@
       </material>
     </visual>
-    <collision>
+    <!-- <collision>
       <origin
         xyz="0 0 0"
@@ -148,5 +147,5 @@
           filename="package://lh_robothand_a0_description/meshes/LF2_Link.STL" />
       </geometry>
-    </collision>
+    </collision> -->
   </link>
   <joint
@@ -205,5 +204,5 @@
       </material>
     </visual>
-    <collision>
+    <!-- <collision>
       <origin
         xyz="0 0 0"
@@ -213,5 +212,5 @@
           filename="package://lh_robothand_a0_description/meshes/LF3_Link.STL" />
       </geometry>
-    </collision>
+    </collision> -->
   </link>
   <joint
@@ -266,5 +265,5 @@
       </material>
     </visual>
-    <collision>
+    <!-- <collision>
       <origin
         xyz="0 0 0"
@@ -274,5 +273,5 @@
           filename="package://lh_robothand_a0_description/meshes/RF1_Link.STL" />
       </geometry>
-    </collision>
+    </collision> -->
   </link>
   <joint
@@ -331,5 +330,5 @@
       </material>
     </visual>
-    <collision>
+    <!-- <collision>
       <origin
         xyz="0 0 0"
@@ -339,5 +338,5 @@
           filename="package://lh_robothand_a0_description/meshes/RF2_Link.STL" />
       </geometry>
-    </collision>
+    </collision> -->
   </link>
   <joint
@@ -396,5 +395,5 @@
       </material>
     </visual>
-    <collision>
+    <!-- <collision>
       <origin
         xyz="0 0 0"
@@ -404,5 +403,5 @@
           filename="package://lh_robothand_a0_description/meshes/RF3_Link.STL" />
       </geometry>
-    </collision>
+    </collision> -->
   </link>
   <joint
@@ -457,5 +456,5 @@
       </material>
     </visual>
-    <collision>
+    <!-- <collision>
       <origin
         xyz="0 0 0"
@@ -465,5 +464,5 @@
           filename="package://lh_robothand_a0_description/meshes/MF1_Link.STL" />
       </geometry>
-    </collision>
+    </collision> -->
   </link>
   <joint
@@ -522,5 +521,5 @@
       </material>
     </visual>
-    <collision>
+    <!-- <collision>
       <origin
         xyz="0 0 0"
@@ -530,5 +529,5 @@
           filename="package://lh_robothand_a0_description/meshes/MF2_Link.STL" />
       </geometry>
-    </collision>
+    </collision> -->
   </link>
   <joint
@@ -587,5 +586,5 @@
       </material>
     </visual>
-    <collision>
+    <!-- <collision>
       <origin
         xyz="0 0 0"
@@ -595,5 +594,5 @@
           filename="package://lh_robothand_a0_description/meshes/MF3_Link.STL" />
       </geometry>
-    </collision>
+    </collision> -->
   </link>
   <joint
@@ -648,5 +647,5 @@
       </material>
     </visual>
-    <collision>
+    <!-- <collision>
       <origin
         xyz="0 0 0"
@@ -656,5 +655,5 @@
           filename="package://lh_robothand_a0_description/meshes/FF1_Link.STL" />
       </geometry>
-    </collision>
+    </collision> -->
   </link>
   <joint
@@ -713,5 +712,5 @@
       </material>
     </visual>
-    <collision>
+    <!-- <collision>
       <origin
         xyz="0 0 0"
@@ -721,5 +720,5 @@
           filename="package://lh_robothand_a0_description/meshes/FF2_Link.STL" />
       </geometry>
-    </collision>
+    </collision> -->
   </link>
   <joint
@@ -778,5 +777,5 @@
       </material>
     </visual>
-    <collision>
+    <!-- <collision>
       <origin
         xyz="0 0 0"
@@ -786,5 +785,5 @@
           filename="package://lh_robothand_a0_description/meshes/FF3_Link.STL" />
       </geometry>
-    </collision>
+    </collision> -->
   </link>
   <joint
@@ -839,5 +838,5 @@
       </material>
     </visual>
-    <collision>
+    <!-- <collision>
       <origin
         xyz="0 0 0"
@@ -847,5 +846,5 @@
           filename="package://lh_robothand_a0_description/meshes/TH1_Link.STL" />
       </geometry>
-    </collision>
+    </collision> -->
   </link>
   <joint
@@ -904,5 +903,5 @@
       </material>
     </visual>
-    <collision>
+    <!-- <collision>
       <origin
         xyz="0 0 0"
@@ -912,5 +911,5 @@
           filename="package://lh_robothand_a0_description/meshes/TH2_Link.STL" />
       </geometry>
-    </collision>
+    </collision> -->
   </link>
   <joint
@@ -969,5 +968,5 @@
       </material>
     </visual>
-    <collision>
+    <!-- <collision>
       <origin
         xyz="0 0 0"
@@ -977,5 +976,5 @@
           filename="package://lh_robothand_a0_description/meshes/TH3_Link.STL" />
       </geometry>
-    </collision>
+    </collision> -->
   </link>
   <joint

File: rh_robothand_a0_description/urdf/rh_robothand_a0.urdf (robot description, URDF)
Before this commit: robot rh_robothand_a0, 16 links, 15 joints
Links:
- link rh_FF1_Link: geometry visual mesh filename=package://rh_robothand_a0_description/meshes/FF1_Link.STL
- link rh_FF2_Link: geometry visual mesh filename=package://rh_robothand_a0_description/meshes/FF2_Link.STL
- link rh_FF3_Link: geometry visual mesh filename=package://rh_robothand_a0_description/meshes/FF3_Link.STL
- link rh_LF1_Link: geometry visual mesh filename=package://rh_robothand_a0_description/meshes/LF1_Link.STL
- link rh_LF2_Link: geometry visual mesh filename=package://rh_robothand_a0_description/meshes/LF2_Link.STL
- link rh_LF3_Link: geometry visual mesh filename=package://rh_robothand_a0_description/meshes/LF3_Link.STL
- link rh_MF1_Link: geometry visual mesh filename=package://rh_robothand_a0_description/meshes/MF1_Link.STL
- link rh_MF2_Link: geometry visual mesh filename=package://rh_robothand_a0_description/meshes/MF2_Link.STL
- link rh_MF3_Link: geometry visual mesh filename=package://rh_robothand_a0_description/meshes/MF3_Link.STL
- link rh_RF1_Link: geometry visual mesh filename=package://rh_robothand_a0_description/meshes/RF1_Link.STL
- link rh_RF2_Link: geometry visual mesh filename=package://rh_robothand_a0_description/meshes/RF2_Link.STL
- link rh_RF3_Link: geometry visual mesh filename=package://rh_robothand_a0_description/meshes/RF3_Link.STL
- link rh_TH1_Link: geometry visual mesh filename=package://rh_robothand_a0_description/meshes/TH1_Link.STL
- link rh_TH2_Link: geometry visual mesh filename=package://rh_robothand_a0_description/meshes/TH2_Link.STL
- link rh_TH3_Link: geometry visual mesh filename=package://rh_robothand_a0_description/meshes/TH3_Link.STL
- link rh_base_link: geometry collision box size=0.22 0.08 0.05; visual mesh filename=package://rh_robothand_a0_description/meshes/base_link.STL

File: rh_robothand_a0_description/urdf/rh_robothand_a0.xacro (robot description, xacro)
@@ -37,9 +37,8 @@
     <collision>
       <origin
-        xyz="0 0 0"
-        rpy="0 0 0" />
-      <geometry>
-        <mesh
-          filename="package://rh_robothand_a0_description/meshes/base_link.STL" />
+        xyz="-0.11 0 0"
+        rpy="0 0 0" />
+      <geometry>
+        <box size="0.22 0.08 0.05"/>
       </geometry>
     </collision>
@@ -75,5 +74,5 @@
       </material>
     </visual>
-    <collision>
+    <!-- <collision>
       <origin
         xyz="0 0 0"
@@ -83,5 +82,5 @@
           filename="package://rh_robothand_a0_description/meshes/LF1_Link.STL" />
       </geometry>
-    </collision>
+    </collision> -->
   </link>
   <joint
@@ -140,5 +139,5 @@
       </material>
     </visual>
-    <collision>
+    <!-- <collision>
       <origin
         xyz="0 0 0"
@@ -148,5 +147,5 @@
           filename="package://rh_robothand_a0_description/meshes/LF2_Link.STL" />
       </geometry>
-    </collision>
+    </collision> -->
   </link>
   <joint
@@ -205,5 +204,5 @@
       </material>
     </visual>
-    <collision>
+    <!-- <collision>
       <origin
         xyz="0 0 0"
@@ -213,5 +212,5 @@
           filename="package://rh_robothand_a0_description/meshes/LF3_Link.STL" />
       </geometry>
-    </collision>
+    </collision> -->
   </link>
   <joint
@@ -266,5 +265,5 @@
       </material>
     </visual>
-    <collision>
+    <!-- <collision>
       <origin
         xyz="0 0 0"
@@ -274,5 +273,5 @@
           filename="package://rh_robothand_a0_description/meshes/RF1_Link.STL" />
       </geometry>
-    </collision>
+    </collision> -->
   </link>
   <joint
@@ -331,5 +330,5 @@
       </material>
     </visual>
-    <collision>
+    <!-- <collision>
       <origin
         xyz="0 0 0"
@@ -339,5 +338,5 @@
           filename="package://rh_robothand_a0_description/meshes/RF2_Link.STL" />
       </geometry>
-    </collision>
+    </collision> -->
   </link>
   <joint
@@ -396,5 +395,5 @@
       </material>
     </visual>
-    <collision>
+    <!-- <collision>
       <origin
         xyz="0 0 0"
@@ -404,5 +403,5 @@
           filename="package://rh_robothand_a0_description/meshes/RF3_Link.STL" />
       </geometry>
-    </collision>
+    </collision> -->
   </link>
   <joint
@@ -457,5 +456,5 @@
       </material>
     </visual>
-    <collision>
+    <!-- <collision>
       <origin
         xyz="0 0 0"
@@ -465,5 +464,5 @@
           filename="package://rh_robothand_a0_description/meshes/MF1_Link.STL" />
       </geometry>
-    </collision>
+    </collision> -->
   </link>
   <joint
@@ -522,5 +521,5 @@
       </material>
     </visual>
-    <collision>
+    <!-- <collision>
       <origin
         xyz="0 0 0"
@@ -530,5 +529,5 @@
           filename="package://rh_robothand_a0_description/meshes/MF2_Link.STL" />
       </geometry>
-    </collision>
+    </collision> -->
   </link>
   <joint
@@ -587,5 +586,5 @@
       </material>
     </visual>
-    <collision>
+    <!-- <collision>
       <origin
         xyz="0 0 0"
@@ -595,5 +594,5 @@
           filename="package://rh_robothand_a0_description/meshes/MF3_Link.STL" />
       </geometry>
-    </collision>
+    </collision> -->
   </link>
   <joint
@@ -648,5 +647,5 @@
       </material>
     </visual>
-    <collision>
+    <!-- <collision>
       <origin
         xyz="0 0 0"
@@ -656,5 +655,5 @@
           filename="package://rh_robothand_a0_description/meshes/FF1_Link.STL" />
       </geometry>
-    </collision>
+    </collision> -->
   </link>
   <joint
@@ -713,5 +712,5 @@
       </material>
     </visual>
-    <collision>
+    <!-- <collision>
       <origin
         xyz="0 0 0"
@@ -721,5 +720,5 @@
           filename="package://rh_robothand_a0_description/meshes/FF2_Link.STL" />
       </geometry>
-    </collision>
+    </collision> -->
   </link>
   <joint
@@ -778,5 +777,5 @@
       </material>
     </visual>
-    <collision>
+    <!-- <collision>
       <origin
         xyz="0 0 0"
@@ -786,5 +785,5 @@
           filename="package://rh_robothand_a0_description/meshes/FF3_Link.STL" />
       </geometry>
-    </collision>
+    </collision> -->
   </link>
   <joint
@@ -839,5 +838,5 @@
       </material>
     </visual>
-    <collision>
+    <!-- <collision>
       <origin
         xyz="0 0 0"
@@ -847,5 +846,5 @@
           filename="package://rh_robothand_a0_description/meshes/TH1_Link.STL" />
       </geometry>
-    </collision>
+    </collision> -->
   </link>
   <joint
@@ -904,5 +903,5 @@
       </material>
     </visual>
-    <collision>
+    <!-- <collision>
       <origin
         xyz="0 0 0"
@@ -912,5 +911,5 @@
           filename="package://rh_robothand_a0_description/meshes/TH2_Link.STL" />
       </geometry>
-    </collision>
+    </collision> -->
   </link>
   <joint
@@ -969,5 +968,5 @@
       </material>
     </visual>
-    <collision>
+    <!-- <collision>
       <origin
         xyz="0 0 0"
@@ -977,5 +976,5 @@
           filename="package://rh_robothand_a0_description/meshes/TH3_Link.STL" />
       </geometry>
-    </collision>
+    </collision> -->
   </link>
   <joint
